File: LNA/LNA.kicad_sch (KiCad schematic)
At the start: 0 parts

Commit message: Add .gitignore and update KiCad project files
Parts:
- added C1, C2: 22uF (16V), symbol Device:C_Polarized_US
- added C3, C4, C5: 100pF, symbol Device:C
- added C6: 10nF, symbol Device:C
- added C7: 100nF, symbol Device:C
- added C8: 1uF, symbol Device:C
- added D1, D2: SS34, Package_TO_SOT_SMD:SOT-363_SC-70-6, symbol Device:D_Schottky
- added D3: PESD5V0U1BL, Package_SON:WSON-6-1EP_2x2mm_P0.65mm_EP1x1.6mm, symbol Device:D_TVS
- added J1, J2: SMA 50R, symbol Connector:Conn_Coaxial
- added J3: DC IN (7-10V), symbol Connector:Screw_Terminal_01x02
- added L1: 10uH, symbol Device:L
- added L2: 330nH - 1uH, symbol Device:L
- added R1, R2: 39R, symbol Device:R
- added U1: SPF5189Z, Package_TO_SOT_SMD:SOT-89-3_Handsoldering, symbol RF_Amplifier:SPF5189Z
- added U2: AMS1117-5.0, Package_TO_SOT_SMD:SOT-223-3_TabPin2, symbol Regulator_Linear:AMS1117-5.0
Connections:
- new net: C5.1, C6.1, C7.1, L1.1, R1.2, R2.2
- new net: C8.1, L1.2, L2.1
- new net: C3.1, D3.2 (A2), J1.1 (In)
- new net: D1.2 (A), J3.1 (Pin_1)
- new net: C1.1, D1.1 (K), U2.3 (VI)
- new net: C2.1, R1.1, R2.1, U2.2 (VO)
- new net: C4.1, L2.2, U1.3
- new net: C3.2, U1.1
- new net: C4.2, J2.1 (In)
- new net GND: C1.2, C2.2, C5.2, C6.2, C7.2, C8.2, D2.2 (A), D3.1 (A1), J1.2 (Ext), J2.2 (Ext), J3.2 (Pin_2), U1.2 (GND), U2.1 (GND)

Commit message: commit
Connections:
- net at D2.1 (K): now also D1.2 (A), J3.1 (Pin_1)

Commit message: completed schematic, now onto routing
Parts:
- C1, C2: footprint (none) -> Capacitor_Tantalum_SMD:CP_EIA-3528-21_Kemet-B_HandSolder
- C3, C4: value 100pF -> 1nF; footprint (none) -> Capacitor_SMD:C_0603_1608Metric_Pad1.08x0.95mm_HandSolder
- C5, C6, C7, C8: footprint (none) -> Capacitor_SMD:C_0603_1608Metric_Pad1.08x0.95mm_HandSolder
- D1, D2: footprint Package_TO_SOT_SMD:SOT-363_SC-70-6 -> Diode_SMD:D_SMA_Handsoldering
- J1, J2: footprint (none) -> Connector_Coaxial:SMA_Amphenol_132289_EdgeMount
- L1: footprint (none) -> Inductor_SMD:L_1210_3225Metric
- L2: footprint (none) -> Inductor_SMD:L_0805_2012Metric
- R1, R2: footprint (none) -> Resistor_SMD:R_0805_2012Metric_Pad1.20x1.40mm_HandSolder
Other:
- note added: "NorthernStudios LNA"
Changed lines of the file:
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@@
 	(generator_version "10.0")
 	(paper "A4")
+	(text "NorthernStudios LNA"
+		(exclude_from_sim no)
+		(at 227.584 175.006 0)
+		(effects
+			(font
+				(size 2.54 2.54)
+				(thickness 0.508)
+				(bold yes)
+				(italic yes)
+			)
+		)
+	)
 	(junction
 		(at 118.11 99.06)
@@
 			)
 		)
-		(property "Footprint" ""
+		(property "Footprint" "Inductor_SMD:L_1210_3225Metric"
 			(at 208.28 100.33 0)
 			(hide yes)
@@
 			)
 		)
-		(property "Footprint" "Package_TO_SOT_SMD:SOT-363_SC-70-6"
+		(property "Footprint" "Diode_SMD:D_SMA_Handsoldering"
 			(at 53.34 106.68 0)
 			(hide yes)
@@
 			)
 		)
-		(property "Footprint" "Package_TO_SOT_SMD:SOT-363_SC-70-6"
+		(property "Footprint" "Diode_SMD:D_SMA_Handsoldering"
 			(at 60.96 99.06 0)
 			(hide yes)
@@
 			)
 		)
-		(property "Footprint" ""
+		(property "Footprint" "Capacitor_SMD:C_0603_1608Metric_Pad1.08x0.95mm_HandSolder"
 			(at 176.2252 107.95 0)
 			(hide yes)
@@
 			)
 		)
-		(property "Footprint" ""
+		(property "Footprint" "Capacitor_Tantalum_SMD:CP_EIA-3528-21_Kemet-B_HandSolder"
 			(at 118.11 102.87 0)
 			(hide yes)
@@
 			)
 		)
-		(property "Footprint" ""
+		(property "Footprint" "Inductor_SMD:L_0805_2012Metric"
 			(at 177.8 68.58 0)
 			(hide yes)
@@
 			)
 		)
-		(property "Footprint" ""
+		(property "Footprint" "Resistor_SMD:R_0805_2012Metric_Pad1.20x1.40mm_HandSolder"
 			(at 139.7 98.298 90)
 			(hide yes)
@@
 			)
 		)
-		(property "Footprint" ""
+		(property "Footprint" "Capacitor_SMD:C_0603_1608Metric_Pad1.08x0.95mm_HandSolder"
 			(at 160.9852 107.95 0)
 			(hide yes)
@@
 			)
 		)
-		(property "Footprint" ""
+		(property "Footprint" "Capacitor_Tantalum_SMD:CP_EIA-3528-21_Kemet-B_HandSolder"
 			(at 76.2 102.87 0)
 			(hide yes)
@@
 			)
 		)
-		(property "Value" "100pF"
+		(property "Value" "1nF"
 			(at 143.51 41.91 90)
 			(show_name no)
@@
 			)
 		)
-		(property "Footprint" ""
+		(property "Footprint" "Capacitor_SMD:C_0603_1608Metric_Pad1.08x0.95mm_HandSolder"
 			(at 147.32 46.0248 0)
 			(hide yes)
@@
 			)
 		)
-		(property "Footprint" ""
+		(property "Footprint" "Connector_Coaxial:SMA_Amphenol_132289_EdgeMount"
 			(at 209.55 46.99 0)
 			(hide yes)
@@
 			)
 		)
-		(property "Value" "100pF"
+		(property "Value" "1nF"
 			(at 185.42 41.91 90)
 			(show_name no)
@@
 			)
 		)
-		(property "Footprint" ""
+		(property "Footprint" "Capacitor_SMD:C_0603_1608Metric_Pad1.08x0.95mm_HandSolder"
 			(at 189.23 46.0248 0)
 			(hide yes)
@@
 			)
 		)
-		(property "Footprint" ""
+		(property "Footprint" "Capacitor_SMD:C_0603_1608Metric_Pad1.08x0.95mm_HandSolder"
 			(at 190.1952 107.95 0)
 			(hide yes)
@@
 			)
 		)
-		(property "Footprint" ""
+		(property "Footprint" "Capacitor_SMD:C_0603_1608Metric_Pad1.08x0.95mm_HandSolder"
 			(at 230.8352 83.82 0)
 			(hide yes)
@@
 			)
 		)
-		(property "Footprint" ""
+		(property "Footprint" "Connector_Coaxial:SMA_Amphenol_132289_EdgeMount"
 			(at 121.92 46.99 0)
 			(hide yes)
@@
 			)
 		)
-		(property "Footprint" ""
+		(property "Footprint" "Resistor_SMD:R_0805_2012Metric_Pad1.20x1.40mm_HandSolder"
 			(at 139.7 103.378 90)
 			(hide yes)

Commit message: finished routing
Parts:
- removed C8: 1uF, Capacitor_SMD:C_0603_1608Metric_Pad1.08x0.95mm_HandSolder, symbol Device:C
- removed L2: 330nH - 1uH, Inductor_SMD:L_0805_2012Metric, symbol Device:L
- D3: footprint Package_SON:WSON-6-1EP_2x2mm_P0.65mm_EP1x1.6mm -> Diode_SMD:D_SOD-882
- J3: footprint (none) -> TerminalBlock:TerminalBlock_MaiXu_MX126-5.0-02P_1x02_P5.00mm
- L1: value 10uH -> 470nH-1uH; footprint Inductor_SMD:L_1210_3225Metric -> Inductor_SMD:L_0805_2012Metric
Connections:
- net at L1.2: now also C4.1, U1.3
Other:
- moved on the sheet: L1
